Commit message: Update 09-Robot_arm.urdf

File: Robotic_arm_modelmake/urdf_tutorial/urdf/09-Robot_arm.urdf (robot description, URDF)
Before this commit: robot Robotarm, 8 links, 7 joints
Joints:
- joint joint_to_Arm1: limit (none) -> lower=-3 upper=0.05 effort=1000.0 velocity=0.5; type continuous -> revolute
- joint joint_to_Arm2: limit (none) -> lower=-2.25 upper=3 effort=1000.0 velocity=0.5; type continuous -> revolute
- joint joint_to_Arm3: limit (none) -> lower=-2.6 upper=2.25 effort=1000.0 velocity=0.5; type continuous -> revolute
- joint joint_to_DOF1: origin xyz=0 0 0.21740000128 -> xyz=0 0 0.16740000128

Commit message: Update 09-Robot_arm.urdf

File: Robotic_arm_modelmake/urdf_tutorial/urdf/09-Robot_arm.urdf (robot description, URDF)
Before this commit: robot Robotarm, 8 links, 7 joints
Links:
- link Arm_box1: geometry collision box size=0.109253 0.09036 0.06535; visual box size=0.109253 0.09036 0.06535
- link Arm_box2: geometry collision box size=0.109253 0.09036 0.06535; visual box size=0.109253 0.09036 0.06535
- link Arm_box3: geometry collision box size=0.109253 0.09036 0.06535; visual box size=0.109253 0.09036 0.06535
Joints:
- joint joint_to_Arm_box1: origin xyz=0 0 0.05 -> xyz=0 0 0.04448

Commit message: Update 09-Robot_arm.urdf

File: Robotic_arm_modelmake/urdf_tutorial/urdf/09-Robot_arm.urdf (robot description, URDF)
Before this commit: robot Robotarm, 8 links, 7 joints
Joints:
- joint joint_to_Arm1: limit lower=-3 upper=0.05 effort=1000.0 velocity=0.5 -> lower=-2.26893 upper=0 effort=1000.0 velocity=0.5
- joint joint_to_Arm2: limit lower=-2.25 upper=3 effort=1000.0 velocity=0.5 -> lower=-0.698132 upper=1.5708 effort=1000.0 velocity=0.5
- joint joint_to_Arm3: limit lower=-2.6 upper=2.25 effort=1000.0 velocity=0.5 -> lower=-0.698132 upper=1.5708 effort=1000.0 velocity=0.5
- joint joint_to_DOF1: limit (none) -> lower=-3.14 upper=3.14 effort=1000.0 velocity=0.5; type continuous -> revolute
